File: recruitment.kicad_sch (KiCad schematic)
At the start: 0 parts

Commit message: Add hierarchical labels and sheet pins
Other:
- added sheet Analog (analog.kicad_sch)
- added sheet Inputs (inputs.kicad_sch)
- added sheet Logic (logic.kicad_sch)
- added sheet Output (output.kicad_sch)
- added sheet Power (power.kicad_sch)
