File: recruitment.kicad_sch (KiCad schematic)
At the start: 0 parts

Commit message: wiring v 1.0
Parts:
- added J1, J4: Conn_01x02, Connector_Molex:Molex_Micro-Fit_3.0_43650-0200_1x02_P3.00mm_Horizontal, symbol Connector_Generic:Conn_01x02
- added J2, J3: Conn_01x03, Connector_Molex:Molex_Micro-Fit_3.0_43650-0315_1x03_P3.00mm_Vertical, symbol Connector_Generic:Conn_01x03
Connections:
- net Analog/+5V: now also J2.3 (Pin_3), J3.3 (Pin_3)
- net Inputs/BRAKE_IN: now also J2.1 (Pin_1)
- net Inputs/PWR_IN: now also J3.1 (Pin_1)
- net Output/SDC: now also J4.1 (Pin_1)
- net Power/VIN: now also J1.1 (Pin_1)
- new net GND: J1.2 (Pin_2), J2.2 (Pin_2), J3.2 (Pin_2), J4.2 (Pin_2)

Commit message: wiring v 1.1
Connections:
- net Analog/+5V: no longer J2.3 (Pin_3), J3.3 (Pin_3)
- net Inputs/BRAKE_IN: now also J2.3 (Pin_3); no longer J2.1 (Pin_1)
- net Inputs/PWR_IN: now also J3.3 (Pin_3); no longer J3.1 (Pin_1)
- new net Inputs/+5V_OUT: J2.1 (Pin_1), J3.1 (Pin_1)
Other:
- sheet Inputs ports: added +5V_OUT; removed none
- moved on the sheet: J2, J3

Commit message: modified connector
Parts:
- removed J1, J4: Conn_01x02, Connector_Molex:Molex_Micro-Fit_3.0_43650-0200_1x02_P3.00mm_Horizontal, symbol Connector_Generic:Conn_01x02
- removed J2, J3: Conn_01x03, Connector_Molex:Molex_Micro-Fit_3.0_43650-0315_1x03_P3.00mm_Vertical, symbol Connector_Generic:Conn_01x03
- added J1, J4: 43650-0201, 43650-02(00,01,02), symbol SamacSys:43650-0201
- added J2, J3: 43650-0301, 43650-03YY, symbol SamacSys:43650-0301
Connections:
- net GND: now also J1.2, J2.2, J3.2, J4.2
- net Inputs/+5V_OUT: now also J2.1, J3.1
- net Inputs/BRAKE_IN: now also J2.3
- net Inputs/PWR_IN: now also J3.3
- net Output/SDC: now also J4.1
- net Power/VIN: now also J1.1

Commit message: Power section finished
Other:
- sheet Power ports: added +5V; removed +5v
Changed lines of the file:
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@@
 			)
 		)
-		(pin "+5v" output
+		(pin "+5V" output
 			(at 92.71 76.2 0)
 			(effects

Commit message: timer doc, simulation and scheme
Other:
- sheet Analog ports: added SENSOR_OK; removed SNS_FAULT
- sheet Logic ports: added SENSOR_OK; removed SNS_FAULT
Changed lines of the file:
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@@
 			)
 		)
-		(pin "SNS_FAULT" output
+		(pin "SENSOR_OK" output
 			(at 139.7 88.9 0)
 			(effects
@@
 			)
 		)
-		(pin "SNS_FAULT" input
+		(pin "SENSOR_OK" input
 			(at 153.67 88.9 180)
 			(effects
