File: recruitment.kicad_sch (KiCad schematic)
At the start: 4 parts, among them J1 43650-0201, J2 43650-0301, J3 43650-0301, J4 43650-0201

Commit message: Latch and reset started
Connections:
- net GND: no longer J4.2
- net Output/SDC renamed Output/SDC_IN
- new net Output/SDC_OUT: J4.2
Other:
- sheet Output ports: added SDC_IN, SDC_OUT; removed SDC
- moved on the sheet: J4
Changed lines of the file:
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@@
-	(wire
-		(pts
-			(xy 233.68 121.92) (xy 237.49 121.92)
-		)
-		(stroke
-			(width 0)
-			(type default)
-		)
-	)
 	(wire
 		(pts
 			(xy 99.06 45.72) (xy 213.36 45.72)
-		)
-		(stroke
-			(width 0)
-			(type default)
-		)
-	)
-	(wire
-		(pts
-			(xy 228.6 124.46) (xy 237.49 124.46)
 		)
 		(stroke
@@
 	(symbol
 		(lib_id "SamacSys:43650-0201")
-		(at 237.49 121.92 0)
+		(at 228.6 121.92 0)
 		(unit 1)
 		(body_style 1)
@@
 		(fields_autoplaced yes)
 		(property "Reference" "J4"
-			(at 254 121.9199 0)
+			(at 245.11 121.9199 0)
 			(show_name no)
 			(do_not_autoplace no)
@@
 		)
 		(property "Value" "43650-0201"
-			(at 254 124.4599 0)
+			(at 245.11 124.4599 0)
 			(show_name no)
 			(do_not_autoplace no)
@@
 		)
 		(property "Footprint" "43650-02(00,01,02)"
-			(at 254 216.84 0)
+			(at 245.11 216.84 0)
 			(hide yes)
 			(show_name no)
@@
 		)
 		(property "Datasheet" "https://www.molex.com/pdm_docs/sd/436500200_sd.pdf"
-			(at 254 316.84 0)
+			(at 245.11 316.84 0)
 			(hide yes)
 			(show_name no)
@@
 		)
 		(property "Description" "Micro-Fit 3.0 Right-Angle Header, 3.00mm Pitch, Single Row, 2 Circuits, with Snap-in Plastic Peg PCB Lock, Glow-Wire Capable, Black"
-			(at 237.49 121.92 0)
+			(at 228.6 121.92 0)
 			(hide yes)
 			(show_name no)
@@
 		)
 		(property "Height" "5.57"
-			(at 254 516.84 0)
+			(at 245.11 516.84 0)
 			(hide yes)
 			(show_name no)
@@
 		)
 		(property "Mouser Part Number" "538-43650-0201"
-			(at 254 616.84 0)
+			(at 245.11 616.84 0)
 			(hide yes)
 			(show_name no)
@@
 		)
 		(property "Mouser Price/Stock" "https://www.mouser.co.uk/ProductDetail/Molex/43650-0201?qs=HlEFOAM0q6XDqOKWr68Eiw%3D%3D"
-			(at 254 716.84 0)
+			(at 245.11 716.84 0)
 			(hide yes)
 			(show_name no)
@@
 		)
 		(property "Manufacturer_Name" "Molex"
-			(at 254 816.84 0)
+			(at 245.11 816.84 0)
 			(hide yes)
 			(show_name no)
@@
 		)
 		(property "Manufacturer_Part_Number" "43650-0201"
-			(at 254 916.84 0)
+			(at 245.11 916.84 0)
 			(hide yes)
 			(show_name no)
@@
 	(symbol
 		(lib_id "power:GND")
-		(at 233.68 121.92 270)
-		(unit 1)
-		(body_style 1)
-		(exclude_from_sim no)
-		(in_bom yes)
-		(on_board yes)
-		(in_pos_files yes)
-		(dnp no)
-		(fields_autoplaced yes)
-		(property "Reference" "#PWR04"
-			(at 227.33 121.92 0)
-			(hide yes)
-			(show_name no)
-			(do_not_autoplace no)
-			(effects
-				(font
-					(size 1.27 1.27)
-				)
-			)
-		)
-		(property "Value" "GND"
-			(at 229.87 121.9199 90)
-			(show_name no)
-			(do_not_autoplace no)
-			(effects
-				(font
-					(size 1.27 1.27)
-				)
-				(justify right)
-			)
-		)
-		(property "Footprint" ""
-			(at 233.68 121.92 0)
-			(hide yes)
-			(show_name no)
-			(do_not_autoplace no)
-			(effects
-				(font
-					(size 1.27 1.27)
-				)
-			)
-		)
-		(property "Datasheet" ""
-			(at 233.68 121.92 0)
-			(hide yes)
-			(show_name no)
-			(do_not_autoplace no)
-			(effects
-				(font
-					(size 1.27 1.27)
-				)
-			)
-		)
-		(property "Description" "Power symbol creates a global label with name \"GND\" , ground"
-			(at 233.68 121.92 0)
-			(hide yes)
-			(show_name no)
-			(do_not_autoplace no)
-			(effects
-				(font
-					(size 1.27 1.27)
-				)
-			)
-		)
-		(pin "1"
-		)
-		(instances
-			(project "recruitment"
-				(path "/bdc7face-9f7c-4701-80bb-4cc144448db1"
-					(reference "#PWR04")
-					(unit 1)
-				)
-			)
-		)
-	)
-	(symbol
-		(lib_id "power:GND")
 		(at 46.99 111.76 90)
 		(unit 1)
@@
 			)
 		)
-		(pin "SDC" output
+		(pin "SDC_IN" output
 			(at 228.6 124.46 0)
 			(effects
 				(font
+					(size 1.27 1.27)
+				)
+				(justify right)
+			)
+		)
+		(pin "SDC_OUT" output
+			(at 228.6 121.92 0)
+			(effects
+				(font

Commit message: output block kicad + docs finished
Other:
- sheet Logic ports: added RELAY_EN; removed BSPD_OK
- sheet Output ports: added RELAY_EN; removed BSPD_OK
Changed lines of the file:
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@@
 			)
 		)
-		(pin "BSPD_OK" output
+		(pin "RELAY_EN" output
 			(at 184.15 127 0)
 			(effects
@@
 			)
 		)
-		(pin "BSPD_OK" input
+		(pin "RELAY_EN" input
 			(at 198.12 127 180)
 			(effects
