File: power.kicad_sch (KiCad schematic)
At the start: 0 parts

Commit message: Power section completed(circuit + docs)
Parts:
- added C1: 100u 50V, Capacitor_SMD:CP_Elec_8x10, symbol Device:C_Polarized
- added C2: C, Capacitor_SMD:C_1206_3216Metric, symbol Device:C
- added C3: 1u, symbol Device:C
- added C4: 0.001u, symbol Device:C
- added C5: 0.1u, symbol Device:C
- added D1: SMBJ18A-E3_5B, DIOM5436X244N, symbol SamacSys:SMBJ18A-E3_5B
- added IC1: LT8607EMSE#PBF, SOP50P490X110-11N, symbol SamacSys:LT8607EMSE#PBF
- added L1: XFL4020-472MEC, XFL4020472MEC, symbol SamacSys:XFL4020-472MEC
- added R1: 18.2k, symbol Device:R_US
- added R2: 1M, Resistor_SMD:R_0603_1608Metric, symbol Device:R_US
- added R3: 184k, Resistor_SMD:R_0603_1608Metric, symbol Device:R_US
Connections:
- net VIN: now also C1.1, C2.1, D1.1 (K), IC1.10 (EN/UV), IC1.9 (VIN)
- new net: C3.2, IC1.3 (INTVCC)
- new net: C5.2, IC1.2 (SW), L1.1
- new net: L1.2, R2.1
- new net: C4.1, IC1.7 (TR/SS)
- new net: C5.1, IC1.1 (BST)
- new net: IC1.4 (RT), R1.1
- new net: IC1.6 (FB), R2.2, R3.1
- new net GND: C1.2, C2.2, C3.1, C4.2, D1.2 (A), IC1.5 (SYNC), R1.2, R3.2
Other:
- note added: "Formula: C1 ≥ 4 × C2, Z0 = √(L_cable / C2) Data: L_cable = 1 µH, C2 = 4.7 µF, V_TVS(clamp) = 29.2 V Resolution: C1 ≥ 4 × 4.7 µF = 19 µF Z0 = sqrt(1 µH / 4.7 µF) ≈ 0.46 Ω → target ESR Chosen: 100 µF (standard value), rated 50 V"
- note added: "The chosen switching frequency is 2 MHz: it is below the maximum frequency allowed by the buck converter and above the AM radio band. The inductor was chosen according to the datasheet reference design (4.7 µH). FORMULA: ripple = V_OUT / (L × f_SW) × (1 − V_OUT / V_IN(MAX)) (datasheet p. 14) Capacitor charging: I_C = C × V / t I_PEAK = I_C + I_LOAD + ripple / 2 DATA: V_OUT = 5 V V_IN(MAX) = 17 V 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"

Commit message: Power section finished
Parts:
- added C6: 22u, symbol Device:C
- added C7: 10p, symbol Device:C
- added D2: PMEG6020ER,115, PMEG6020ER115, symbol SamacSys:PMEG6020ER,115
- added FB1: BLM18KG601SH1D, BLM18SP221SN1B, symbol SamacSys:BLM18KG601SH1D
- C2: value C -> 4.7u
- C4: value 0.001u -> 1n
- R3: value 184k -> 187k
Connections:
- net +5V_RELAY: now also FB1.2
- net GND: now also IC1.11 (EP), C6.2
- net VIN: now also D2.2 (A); no longer C1.1, C2.1, D1.1 (K), IC1.10 (EN/UV), IC1.9 (VIN)
- net +5V: now reaches L1.2, R2.1
- net +5V: now also C6.1, C7.1, FB1.1
- net at IC1.6 (FB), R2.2, R3.1: now also C7.2
- new net: C1.1, C2.1, D1.1 (K), D2.1 (K), IC1.10 (EN/UV), IC1.9 (VIN)
Other:
- note added: "FORMULA: C1 >> C2, Z0 = √(L_cable / C2) DATA: L_cable = 1 µH, C2 = 4.7 µF, V_TVS(clamp) = 29.2 V RESOLUTION: C1 ≥ 4 × 4.7 µF = 19 µF Z0 = sqrt(1 µH / 4.7 µF) ≈ 0.46 Ω"
- note added: "FORMULA: C_OUT = 100/(V_OUT/f_sw), ΔV_OUT ≈ ΔI_L / (8 × f_SW × C_OUT) DATA: V_OUT = 5V, f_Sw = 2, ΔI_L = 0.38A(inductor ripple current) RESOLUTION: C_OUT = 100 / (5 × 2) C_OUT = 10 µF (at minimum) ΔV_OUT ≈ 0,38 A / (8 × 2 MHz × 22 µF) ΔV_OUT ≈ 1,1 mV"
- note added: "The chosen switching frequency is 2 MHz: it is below the maximum frequency allowed by the buck converter and above the AM radio band. The inductor was chosen according to the datasheet reference design (4.7 µH). FORMULA: ripple = V_OUT / (L × f_SW) × (1 − V_OUT / V_IN(MAX)) (datasheet p. 14) Capacitor charging: I_C = C × V / t I_PEAK = I_C + I_LOAD + ripple / 2 DATA: V_OUT = 5 V, V_IN(MAX) = 17 V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"
- note removed: "Formula: C1 ≥ 4 × C2, Z0 = √(L_cable / C2) Data: L_cable = 1 µH, C2 = 4.7 µF, V_TVS(clamp) = 29.2 V Resolution: C1 ≥ 4 × 4.7 µF = 19 µF Z0 = sqrt(1 µH / 4.7 µF) ≈ 0.46 Ω → target ESR Chosen: 100 µF (standard value), rated 50 V"
- note removed: "The chosen switching frequency is 2 MHz: it is below the maximum frequency allowed by the buck converter and above the AM radio band. The inductor was chosen according to the datasheet reference design (4.7 µH). FORMULA: ripple = V_OUT / (L × f_SW) × (1 − V_OUT / V_IN(MAX)) (datasheet p. 14) Capacitor charging: I_C = C × V / t I_PEAK = I_C + I_LOAD + ripple / 2 DATA: V_OUT = 5 V V_IN(MAX) = 17 V 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"
- moved on the sheet: C1, C2, C3, C4, C5, D1, IC1, L1, R1, R2, R3
