File: power.kicad_sch (KiCad schematic)
At the start: 15 parts, among them IC1 LT8607EMSE#PBF

Commit message: Latch and reset started
Connections:
- no-connect marks 0 -> 2
Changed lines of the file:
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@@
 		(color 0 0 0 0)
+	)
+	(no_connect
+		(at 129.54 49.53)
+	)
+	(no_connect
+		(at 46.99 55.88)
 	)
 	(wire

Commit message: Logic section kicad + docs
Parts:
- added LED2: SMLD12EN1WT86C, SMLD12EN1WT86C, symbol SamacSys:SMLD12EN1WT86C
- added R25: 715, Resistor_SMD:R_0603_1608Metric, symbol Device:R_US
Connections:
- net +5V: now also R25.2
- net GND: now also LED2.1 (K)
- new net: LED2.2 (A), R25.1
