File: inputs.kicad_sch (KiCad schematic)
At the start: 0 parts

Commit message: wiring v 1.1
Changed lines of the file:
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@@
+		)
+	)
+	(hierarchical_label "+5V_OUT"
+		(shape output)
+		(at 76.2 52.07 0)
+		(effects
+			(font
+				(size 1.27 1.27)
+			)
+			(justify left)
 		)
 	)

Commit message: Filter section done
Parts:
- added C8, C9: 100n 50V X7R, Capacitor_SMD:C_0603_1608Metric, symbol Device:C
- added R4, R5: 10k, Resistor_SMD:R_0603_1608Metric, symbol Device:R_US
Connections:
- net BRAKE_FILT: now also C9.1, R5.2
- net BRAKE_IN: now also R5.1
- net PWR_FILT: now also C8.1, R4.2
- net PWR_IN: now also R4.1
- new net GND: C8.2, C9.2
Other:
- note added: "ASSUMPTION: Fastest pedal stomp: 50ms, Inverter's noise: 10kHz Delay: τ = 1ms (5τ = 5ms, 1% of the 500ms) FORMULAS: f = 0.35/t, f_C = 1/(2π*t) RESOLUTION: f = 0.35/0.05s = 7Hz -> 10Hz f_C = 1/(2π*1ms) = 160HZ(teorical)(2π*t) C_F = 100nF(standard) R_TOT = 1/(2π*160 Hz*100 nF) = 9.95kΩ R_IN = 9.95k - 100 = 9.85 -> 10K CONFIRMATION: f_C = 1 / (2π × 10.1 kΩ × 100 nF) = 158HZ"

Commit message: analog block docs and sterted kicad
Parts:
- added R6, R7: 100k, Resistor_SMD:R_0603_1608Metric, symbol Device:R_US
Connections:
- net BRAKE_IN: now also R7.1
- net GND: now also R6.2, R7.2
- net PWR_IN: now also R6.1
