File: inputs.kicad_sch (KiCad schematic)
At the start: 6 parts

Commit message: Latch and reset started
Changed lines of the file:
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@@
 	(wire
 		(pts
-			(xy 124.46 68.58) (xy 181.61 68.58)
+			(xy 123.19 68.58) (xy 181.61 68.58)
 		)
 		(stroke
@@
 	(hierarchical_label "+5V"
 		(shape input)
-		(at 124.46 68.58 180)
+		(at 123.19 68.58 180)
 		(effects
 			(font
