File: analog.kicad_sch (KiCad schematic)
At the start: 0 parts

Commit message: analog block docs and sterted kicad
Parts:
- added R10, R11, R12, R13, R14, R8, R9: R_US, Resistor_SMD:R_0603_1608Metric, symbol Device:R_US
Connections:
- net +5V: now also R10.1, R12.1, R8.1
- new net: R10.2, R11.1
- new net: R13.2, R14.1
- new net: R12.2, R13.1
- new net: R8.2, R9.1
- new net GND: R11.2, R14.2, R9.2
Other:
- note added: "VOLTAGE DIVIDERS (R_TOT ≈ 100 kΩ) FORMULA: R2 = R_TOT × V_REF / 5 V R1 = R_TOT − R2 (R1 to +5V, R2 to GND) RESOLUTION: Brake threshold (V_REF = 1.683 V): R2 = 100 kΩ × 1.683 / 5 = 33.7 kΩ → 34.0 kΩ R1 = 100 kΩ − 33.7 kΩ = 66.3 kΩ → 66.5 kΩ Power threshold (V_REF = 2.640 V max): R2 = 100 kΩ × 2.640 / 5 = 52.8 kΩ → 52.3 kΩ R1 = 100 kΩ − 52.8 kΩ = 47.2 kΩ → 47.5 kΩ Window (V_LOW = 0.25 V, V_HIGH = 4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"

Commit message: Brake-side analog circuit with calculation
Parts:
- added IC2: TLV9024QPWRQ1, SOP65P640X120-14N, symbol SamacSys:TLV9024QPWRQ1
Changed lines of the file:
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@@
+	)
+	(symbol
+		(lib_id "SamacSys:TLV9024QPWRQ1")
+		(at 74.93 36.83 0)
+		(unit 1)
+		(body_style 1)
+		(exclude_from_sim no)
+		(in_bom yes)
+		(on_board yes)
+		(in_pos_files yes)
+		(dnp no)
+		(fields_autoplaced yes)
+		(property "Reference" "IC2"
+			(at 88.9 29.21 0)
+			(show_name no)
+			(do_not_autoplace no)
+			(effects
+				(font
+					(size 1.27 1.27)
+				)
+			)
+		)
+		(property "Value" "TLV9024QPWRQ1"
+			(at 88.9 31.75 0)
+			(show_name no)
+			(do_not_autoplace no)
+			(effects
+				(font
+					(size 1.27 1.27)
+				)
+			)
+		)
+		(property "Footprint" "SOP65P640X120-14N"
+			(at 99.06 131.75 0)
+			(hide yes)
+			(show_name no)
+			(do_not_autoplace no)
+			(effects
+				(font
+					(size 1.27 1.27)
+				)
+				(justify left top)
+			)
+		)
+		(property "Datasheet" "https://www.ti.com/lit/ds/symlink/tlv9024-q1.pdf?ts=1630838462923&ref_url=https%253A%252F%252Fwww.ti.com%252Fstore%252Fti%252Fen%252Fp%252Fproduct%252F%253Fp%253DTLV9024QPWRQ1"
+			(at 99.06 231.75 0)
+			(hide yes)
+			(show_name no)
+			(do_not_autoplace no)
+			(effects
+				(font
+					(size 1.27 1.27)
+				)
+				(justify left top)
+			)
+		)
+		(property "Description" "Automotive, 5.5-V, low-voltage, high-performance, quad open-drain comparator with 120-ns delay"
+			(at 77.216 25.654 0)
+			(hide yes)
+			(show_name no)
+			(do_not_autoplace no)
+			(effects
+				(font
+					(size 1.27 1.27)
+				)
+			)
+		)
+		(property "Height" "1.2"
+			(at 99.06 431.75 0)
+			(hide yes)
+			(show_name no)
+			(do_not_autoplace no)
+			(effects
+				(font
+					(size 1.27 1.27)
+				)
+				(justify left top)
+			)
+		)
+		(property "Mouser Part Number" "595-TLV9024QPWRQ1"
+			(at 99.06 531.75 0)
+			(hide yes)
+			(show_name no)
+			(do_not_autoplace no)
+			(effects
+				(font
+					(size 1.27 1.27)
+				)
+				(justify left top)
+			)
+		)
+		(property "Mouser Price/Stock" "https://www.mouser.co.uk/ProductDetail/Texas-Instruments/TLV9024QPWRQ1?qs=QNEnbhJQKvYmKU2ai0T1Hw%3D%3D"
+			(at 99.06 631.75 0)
+			(hide yes)
+			(show_name no)
+			(do_not_autoplace no)
+			(effects
+				(font
+					(size 1.27 1.27)
+				)
+				(justify left top)
+			)
+		)
+		(property "Manufacturer_Name" "Texas Instruments"
+			(at 99.06 731.75 0)
+			(hide yes)
+			(show_name no)
+			(do_not_autoplace no)
+			(effects
+				(font
+					(size 1.27 1.27)
+				)
+				(justify left top)
+			)
+		)
+		(property "Manufacturer_Part_Number" "TLV9024QPWRQ1"
+			(at 99.06 831.75 0)
+			(hide yes)
+			(show_name no)
+			(do_not_autoplace no)
+			(effects
+				(font
+					(size 1.27 1.27)
+				)
+				(justify left top)
+			)
+		)
+		(pin "13"
+		)
+		(pin "10"
+		)
+		(pin "4"
+		)
+		(pin "1"
+		)
+		(pin "2"
+		)
+		(pin "6"
+		)
+		(pin "12"
+		)
+		(pin "5"
+		)
+		(pin "9"
+		)
+		(pin "14"
+		)
+		(pin "11"
+		)
+		(pin "7"
+		)
+		(pin "8"
+		)
+		(pin "3"
+		)
+		(instances
+			(project "recruitment"
+				(path "/bdc7face-9f7c-4701-80bb-4cc144448db1/30ec489d-3016-4343-8d00-26eafa21f72a"
+					(reference "IC2")
+					(unit 1)
+				)
+			)
+		)
 	)
 	(symbol

Commit message: analog section finished
Parts:
- added C10: 100n, Capacitor_SMD:C_0603_1608Metric, symbol Device:C
- added C11: C, Capacitor_SMD:C_0603_1608Metric, symbol Device:C
- added IC3: TLV9024QPWRQ1, SOP65P640X120-14N, symbol SamacSys:TLV9024QPWRQ1
- added R15, R19, R20, R21: 10k, symbol Device:R_US
- added R16: 1M, symbol Device:R_US
- added R17: 47,5k, symbol Device:R_US
- added R18: 52,3k, symbol Device:R_US
- R10: value R_US -> 10k; footprint Resistor_SMD:R_0603_1608Metric -> (none)
- R11: value R_US -> 1M; footprint Resistor_SMD:R_0603_1608Metric -> (none)
- R12, R14: value R_US -> 4,99k; footprint Resistor_SMD:R_0603_1608Metric -> (none)
- R13: value R_US -> 90,9k; footprint Resistor_SMD:R_0603_1608Metric -> (none)
- R8: value R_US -> 66,5K; footprint Resistor_SMD:R_0603_1608Metric -> (none)
- R9: value R_US -> 34,0K; footprint Resistor_SMD:R_0603_1608Metric -> (none)
Connections:
- net +5V: now also IC2.3 (V+), C10.1, C11.1, IC3.3 (V+), R15.2, R17.1, R20.2, R21.2; no longer R10.1
- net BRAKE_FILT: now also IC2.6 (IN2-), IC2.9 (IN3+), R10.1
- net BRAKE_HIGH: now also IC2.2 (OUT1), R11.2, R15.1
- net GND: now also IC2.12 (V-), C10.2, C11.2, IC3.12 (V-), R18.2; no longer R11.2
- net PWR_FILT: now also IC3.7 (IN2+), IC3.8 (IN3-), R19.1
- net PWR_HIGH: now also IC3.2 (OUT1), R16.2, R20.1
- net at R10.2, R11.1: now also IC2.5 (IN1+)
- net at R13.2, R14.1: now also IC2.8 (IN3-), IC3.6 (IN2-)
- net at R12.2, R13.1: now also IC2.7 (IN2+), IC3.9 (IN3+)
- net at R8.2, R9.1: now also IC2.4 (IN1-)
- net SENSOR_OK: now reaches IC2.1 (OUT2)
- net SENSOR_OK: now also IC2.14 (OUT3), IC3.1 (OUT2), IC3.14 (OUT3), R21.1
- new net: IC3.4 (IN1-), R17.2, R18.1
- new net: IC3.5 (IN1+), R16.1, R19.2
Other:
- note added: "BRAKE_HIGH"
- note added: "Brake_V"
- note added: "FORMULA: ΔV = V_IN * R_S / R_H DATA: V_IN = 4,94V, RS = 10k, R_H = 1M ΔV = 4,94V * 10k/100M = 0.049V = 49mV"
- note added: "VOLTAGE DIVIDERS (R_TOT ≈ 100 kΩ, V_SUPPLY = 4.94 V) FORMULA: R2 = R_TOT × V_REF / 4.94 V R1 = R_TOT − R2 (R1 to +5V, R2 to GND) RESOLUTION: Brake threshold (V_REF = 1.683 V): R2 = 100 kΩ × 1.683 / 4.94 = 34.1 kΩ → 34.0 kΩ R1 = 100 kΩ − 34.1 kΩ = 65.9 kΩ → 66.5 kΩ Check: V_REF = 4.94 × 34.0 / 100.5 = 1.671 V Power threshold (V_REF = 2.640 V max): R2 = 100 kΩ × 2.640 / 4.94 = 53.4 kΩ R1 = 100 kΩ −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"
- note added: "Win_High_V"
- note added: "Win_Low_V"
- note removed: "VOLTAGE DIVIDERS (R_TOT ≈ 100 kΩ) FORMULA: R2 = R_TOT × V_REF / 5 V R1 = R_TOT − R2 (R1 to +5V, R2 to GND) RESOLUTION: Brake threshold (V_REF = 1.683 V): R2 = 100 kΩ × 1.683 / 5 = 33.7 kΩ → 34.0 kΩ R1 = 100 kΩ − 33.7 kΩ = 66.3 kΩ → 66.5 kΩ Power threshold (V_REF = 2.640 V max): R2 = 100 kΩ × 2.640 / 5 = 52.8 kΩ → 52.3 kΩ R1 = 100 kΩ − 52.8 kΩ = 47.2 kΩ → 47.5 kΩ Window (V_LOW = 0.25 V, V_HIGH = 4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"
- moved on the sheet: IC2
