File: analog.kicad_sch (KiCad schematic)
At the start: 18 parts, among them IC2 TLV9024QPWRQ1, IC3 TLV9024QPWRQ1

Commit message: Latch and reset started
Connections:
- net +5V: now also IC2.10 (IN4-), IC3.11 (IN4+)
- net GND: now also IC2.11 (IN4+), IC3.10 (IN4-)
- no-connect marks 0 -> 2
Other:
- moved on the sheet: R17, R18
