File: logic.kicad_sch (KiCad schematic)
At the start: 0 parts

Commit message: timer doc, simulation and scheme
Parts:
- added C12: 1u, Capacitor_SMD:C_1210_3225Metric, symbol Device:C
- added D3: BAS316, Diode_SMD:D_SOD-323, symbol Diode:BAS316
- added IC4: 74AHC1G08GW-Q100,1, SOT65P212X110-5N, symbol SamacSys:74AHC1G08GW-Q100,1
- added IC5: 74HC14PW-Q100,118, SOP65P640X110-14N, symbol SamacSys:74HC14PW-Q100,118
- added R22: 649k, Resistor_SMD:R_0603_1608Metric, symbol Device:R_US
Connections:
- net +5V: now also IC4.5 (VCC), IC5.14 (VCC)
- net BRAKE_HIGH: now also IC4.1 (B)
- net PWR_HIGH: now also IC4.2 (A)
- new net: D3.1 (K), IC4.4 (Y), R22.1
- new net: C12.1, D3.2 (A), IC5.1 (1A), R22.2
- new net GND: C12.2, IC4.3 (GND), IC5.7 (GND)
