File: logic.kicad_sch (KiCad schematic)
At the start: 5 parts, among them IC4 74AHC1G08GW-Q100,1, IC5 74HC14PW-Q100,118

Commit message: Latch and reset started
Parts:
- added IC6: 74AHC1G08GW-Q100,1, SOT65P212X110-5N, symbol SamacSys:74AHC1G08GW-Q100,1
- added IC7, IC8: 74HC1G00GV,125, SOT95P275X110-5N, symbol SamacSys:74HC1G00GV,125
- added R23: R_US, Resistor_SMD:R_0603_1608Metric, symbol Device:R_US
Connections:
- net +5V: now also IC6.5 (VCC), IC7.5 (VCC), IC8.5 (VCC)
- net BSPD_OK: now also IC7.1 (B), IC8.4 (Y)
- net GND: now also IC5.11 (5A), IC5.3 (2A), IC5.5 (3A), IC5.9 (4A), IC6.3 (GND), IC7.3 (GND), IC8.3 (GND), R23.2
- net SENSOR_OK: now also IC6.1 (B)
- net at IC5.12 (6Y): now also IC8.2 (A)
- net at IC5.13 (6A): now also R23.1
- net at IC5.2 (1Y): now also IC6.2 (A)
- new net: IC7.4 (Y), IC8.1 (B)
- new net: IC6.4 (Y), IC7.2 (A)
- no-connect marks 0 -> 4
Other:
- note added: "BSPD_OK"
- note added: "LATCH_FAULT"
- note added: "LATCH_OK"
- note added: "RC TIMER FORMULA: t = τ × ln(V_CC / (V_CC − V_T+)), τ = R × C DATA: V_CC = 4.94 V, V_T+ = 2.60 V (74HC14) t = 485 ms (right, below 500 ms), C = 1 µF RESOLUTION: t = τ × ln(4.94 / 2.34) = 0.75 × τ τ = 0.485 s / 0.75 = 0.65 s R = τ / C = 0.65 s / 1 µF = 650 kΩ → 649 kΩ"
- note added: "READY"
- moved on the sheet: C12, D3, IC4, IC5, R22

Commit message: Logic section kicad + docs
Parts:
- added C13: 1u, Capacitor_SMD:C_1206_3216Metric, symbol Device:C
- added D4: BAS316, Diode_SMD:D_SOD-323, symbol Diode:BAS316
- added LED1: SML-D12L8WT86, SMLD12L8WT86, symbol SamacSys:SML-D12L8WT86
- added LED3, LED4: SML-D12Y1WT86, LEDC1608X55N, symbol SamacSys:SML-D12Y1WT86
- added R24: 1.5k, Resistor_SMD:R_0603_1608Metric, symbol Device:R_US
- added R26, R27: 1.37k, Resistor_SMD:R_0603_1608Metric, symbol Device:R_US
- R23: value R_US -> 100k
Connections:
- net +5V: now also C13.1, R26.2, R27.2
- net BRAKE_HIGH: now also IC5.5 (3A)
- net GND: now also D4.2 (A), LED1.1 (K); no longer IC5.3 (2A), IC5.5 (3A)
- net PWR_HIGH: now also IC5.3 (2A)
- net at IC5.13 (6A), R23.1: now also C13.2, D4.1 (K)
- net at IC7.4 (Y), IC8.1 (B): now also R24.1
- net at IC5.4 (2Y): now also LED3.1 (K)
- net at IC5.6 (3Y): now also LED4.1 (K)
- new net: LED1.2 (A), R24.2
- new net: LED3.2 (A), R26.1
- new net: LED4.2 (A), R27.1
- no-connect marks 4 -> 2
Other:
- note added: "RC TIMER FORMULA: t = τ * ln(V_CC / (V_CC − V_T+)), τ = R * C DATA: V_CC = 4.94 V, V_T+ = 2.60 V (74HC14) t = 485 ms (right, below 500 ms), C = 1 µF RESOLUTION: t = τ * ln(4.94 / 2.34) = 0.75 * τ τ = 0.485 s / 0.75 = 0.65 s R = τ / C = 0.65 s / 1 uF = 650 kΩ -> 649 kΩ"
- note added: "TURN-ON RESET FORMULA: t = τ * ln(V_CC / V_T−), τ = R * C DATA: V_CC = 4.94 V, V_T− = 1.54 V (74HC14) t = 100 ms ( 10 times the settling time), R = 100 kΩ RESOLUTION: t = τ * ln(4.94 / 1.54) = 1.17 × τ τ = 0.1 s / 1.17 = 0.086 s C = τ / R = 0.086 s / 100 kΩ = 0.86 uF -> 1uF"
- note removed: "RC TIMER FORMULA: t = τ × ln(V_CC / (V_CC − V_T+)), τ = R × C DATA: V_CC = 4.94 V, V_T+ = 2.60 V (74HC14) t = 485 ms (right, below 500 ms), C = 1 µF RESOLUTION: t = τ × ln(4.94 / 2.34) = 0.75 × τ τ = 0.485 s / 0.75 = 0.65 s R = τ / C = 0.65 s / 1 µF = 650 kΩ → 649 kΩ"
- moved on the sheet: IC5

Commit message: relay out connection and mosfet connection
Other:
- note added: "START UP RESET FORMULA: t = τ * ln(V_CC / V_T−), τ = R * C DATA: V_CC = 4.94 V, V_T− = 1.54 V (74HC14) t = 100 ms ( 10 times the settling time), R = 100 kΩ RESOLUTION: t = τ * ln(4.94 / 1.54) = 1.17 × τ τ = 0.1 s / 1.17 = 0.086 s C = τ / R = 0.086 s / 100 kΩ = 0.86 uF -> 1uF"
- note removed: "TURN-ON RESET FORMULA: t = τ * ln(V_CC / V_T−), τ = R * C DATA: V_CC = 4.94 V, V_T− = 1.54 V (74HC14) t = 100 ms ( 10 times the settling time), R = 100 kΩ RESOLUTION: t = τ * ln(4.94 / 1.54) = 1.17 × τ τ = 0.1 s / 1.17 = 0.086 s C = τ / R = 0.086 s / 100 kΩ = 0.86 uF -> 1uF"
Changed lines of the file:
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@@
 		)
 	)
-	(text "TURN-ON RESET\nFORMULA:\n  t = τ * ln(V_CC / V_T−),  τ = R * C\nDATA:\n  V_CC = 4.94 V, V_T− = 1.54 V (74HC14)\n  t = 100 ms ( 10 times the settling time), R = 100 kΩ\nRESOLUTION:\n  t = τ * ln(4.94 / 1.54) = 1.17 × τ\n  τ = 0.1 s / 1.17 = 0.086 s\n  C = τ / R = 0.086 s / 100 kΩ = 0.86 uF -> 1uF\n"
+	(text "START UP RESET\nFORMULA:\n  t = τ * ln(V_CC / V_T−),  τ = R * C\nDATA:\n  V_CC = 4.94 V, V_T− = 1.54 V (74HC14)\n  t = 100 ms ( 10 times the settling time), R = 100 kΩ\nRESOLUTION:\n  t = τ * ln(4.94 / 1.54) = 1.17 × τ\n  τ = 0.1 s / 1.17 = 0.086 s\n  C = τ / R = 0.086 s / 100 kΩ = 0.86 uF -> 1uF\n"
 		(exclude_from_sim no)
 		(at 18.542 179.07 0)

Commit message: output block kicad + docs finished
Connections:
- net BSPD_OK renamed RELAY_EN
Changed lines of the file:
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@@
 		)
 	)
-	(hierarchical_label "BSPD_OK"
+	(hierarchical_label "RELAY_EN"
 		(shape output)
 		(at 250.19 119.38 0)
