File: output.kicad_sch (KiCad schematic)
At the start: 0 parts

Commit message: Latch and reset started
Changed lines of the file:
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@@
 		)
 	)
-	(hierarchical_label "SDC"
+	(hierarchical_label "SDC_IN"
+		(shape output)
+		(at 114.3 69.85 0)
+		(effects
+			(font
+				(size 1.27 1.27)
+			)
+			(justify left)
+		)
+	)
+	(hierarchical_label "SDC_OUT"
 		(shape output)
 		(at 114.3 72.39 0)

Commit message: relay out connection and mosfet connection
Parts:
- added K1: TX2SS-5V-X, ATXS20020SS, symbol SamacSys:TX2SS-5V-X
- added LED5: SMLD12EN1WT86C, SMLD12EN1WT86C, symbol SamacSys:SMLD12EN1WT86C
- added Q1: 2N7002BK,215, SOT95P230X110-3N, symbol SamacSys:2N7002BK,215
- added R28: 470, Resistor_SMD:R_0603_1608Metric, symbol Device:R_US
- added R29: 100k, Resistor_SMD:R_0603_1608Metric, symbol Device:R_US
- added R30: 715, Resistor_SMD:R_0603_1608Metric, symbol Device:R_US
Connections:
- net BSPD_OK: now also R28.1, R30.1
- net SDC_IN: now also K1.9 (COM_2)
- net SDC_OUT: now also K1.5 (N.O._1)
- new net: LED5.2 (A), R30.2
- new net: Q1.1 (G), R28.2, R29.1
- new net: K1.4 (COM_1), K1.8 (N.O._2)
- new net GND: LED5.1 (K), Q1.2 (S), R29.2
- no-connect marks 0 -> 2

Commit message: output block kicad + docs finished
Parts:
- added C14: 10u, Capacitor_SMD:C_1206_3216Metric, symbol Device:C
- added C15: 100n, Capacitor_SMD:C_0603_1608Metric, symbol Device:C
- added D5: BAS316, Diode_SMD:D_SOD-323, symbol Diode:BAS316
Connections:
- net +5V_RELAY: now also K1.1 (COIL_+), C14.2, C15.2, D5.1 (K)
- net GND: now also C14.1, C15.1
- net at Q1.3 (D): now also K1.12 (COIL_-), D5.2 (A)
- net BSPD_OK renamed RELAY_EN
Other:
- moved on the sheet: K1, LED5, Q1, R28, R29, R30
